File: hardware/LEDStrip.kicad_sch (KiCad schematic)
At the start: 3 parts, among them J501 WAGO-2065, J502 WAGO-2065, U501 74AHC1G125

Commit message: Replace Order_Number
Parts:
- J501, J502: value WAGO-2065 -> WAGO 2065-100; Manufacturer (none) -> WAGO; Product (none) -> 2065-100/998-403
- U501: footprint Package_TO_SOT_SMD:SOT-23-5 -> V2_Package_TO_SOT_SMD:SOT-23-5; Manufacturer (none) -> Texas Instruments; Mouser (none) -> 595-SN74AHC1G125DBVR; Product (none) -> SN74AHC1G125DBVR
