File: hardware/LEDStrip.kicad_sch (KiCad schematic)
At the start: 3 parts, among them J501 WAGO 2065-100, J502 WAGO 2065-100, U501 74AHC1G125

Commit message: Refresh
Other:
- title: LED Strip -> V2 wave

Commit message: Update
Parts:
- J501, J502: Id (none) -> WAGO:${SYMBOL_NAME}
- U501: Id (none) -> 74xGxx:${SYMBOL_NAME}
Changed lines of the file:
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@@
 	(title_block
 		(title "V2 wave")
-		(date "2026-03-26")
-		(rev "2026-03-11")
+		(date "2026-04-03")
+		(rev "2026-04-03")
 		(company "Versio Duo")
 	)
@@
 			)
 		)
+		(property "Id" "WAGO:${SYMBOL_NAME}"
+			(at 175.26 115.57 0)
+			(hide yes)
+			(show_name no)
+			(do_not_autoplace no)
+			(effects
+				(font
+					(size 1.27 1.27)
+				)
+			)
+		)
 		(pin "1"
 		)
@@
 			)
 		)
+		(property "Id" "WAGO:${SYMBOL_NAME}"
+			(at 175.26 118.11 0)
+			(hide yes)
+			(show_name no)
+			(do_not_autoplace no)
+			(effects
+				(font
+					(size 1.27 1.27)
+				)
+			)
+		)
 		(pin "1"
 		)
@@
 			(hide yes)
 			(show_name no)
+			(do_not_autoplace no)
+			(effects
+				(font
+					(size 1.27 1.27)
+				)
+			)
+		)
+		(property "Id" "74xGxx:${SYMBOL_NAME}"
+			(at 138.43 124.46 0)
+			(hide yes)
+			(show_name no)

Commit message: Update
Parts:
- J501, J502: Rating (none) -> 9A
- U501: Rating (none) -> 8mA
Changed lines of the file:
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@@
 	(title_block
 		(title "V2 wave")
-		(date "2026-04-03")
-		(rev "2026-04-03")
+		(date "2026-04-14")
+		(rev "2026-04-14")
 		(company "Versio Duo")
+		(comment 1 "Power Amplifier")
 	)
 	(junction
@@
 			)
 		)
+		(property "Rating" "9A"
+			(at 175.26 127 0)
+			(hide yes)
+			(show_name no)
+			(do_not_autoplace no)
+			(effects
+				(font
+					(size 1.27 1.27)
+				)
+			)
+		)
 		(pin "1"
 		)
@@
 			)
 		)
+		(property "Rating" "9A"
+			(at 175.26 129.54 0)
+			(hide yes)
+			(show_name no)
+			(do_not_autoplace no)
+			(effects
+				(font
+					(size 1.27 1.27)
+				)
+			)
+		)
 		(pin "1"
 		)
@@
 			(hide yes)
 			(show_name no)
+			(do_not_autoplace no)
+			(effects
+				(font
+					(size 1.27 1.27)
+				)
+			)
+		)
+		(property "Rating" "8mA"
+			(at 138.43 142.24 0)
+			(hide yes)
+			(show_name no)
