File: hardware/wave.kicad_sch (KiCad schematic)
At the start: 62 parts, among them J101 CORTEX-DEBUG, J102 WAGO-2065, J103 WAGO-2065, J104 WAGO-2065, J105 WAGO-2065, J106 WAGO-2065, J107 WAGO-2065, SW101 SW_Push, SW102 SW_Push, U101 TPS78433QWDRBRQ1, U102 ATSAMD51J, Y101 32k768

Commit message: Replace Order_Number
Parts:
- C101: renamed from C109; footprint Capacitor_SMD:C_0603_1608Metric -> V2_Capacitor_SMD:C_0603; symbol Device:C_Small -> V2_Device:C_0603_18p; Manufacturer (none) -> YAGEO; Mouser (none) -> 603-CC603JRNPO9BN180; Product (none) -> CC0603JRNPO9BN180
- C102: renamed from C110; footprint Capacitor_SMD:C_0603_1608Metric -> V2_Capacitor_SMD:C_0603; symbol Device:C_Small -> V2_Device:C_0603_18p; Manufacturer (none) -> YAGEO; Mouser (none) -> 603-CC603JRNPO9BN180; Product (none) -> CC0603JRNPO9BN180
- C103: renamed from C113; footprint Capacitor_SMD:C_0603_1608Metric -> V2_Capacitor_SMD:C_0603; symbol Device:C_Small -> V2_Device:C_0603_0u1; Manufacturer (none) -> TDK; Mouser (none) -> 810-CGA3E2X7R1H104MA; Product (none) -> CGA3E2X7R1H104M080AA; Rating (none) -> 50V
- C104: renamed from C101; footprint Capacitor_SMD:C_0603_1608Metric -> V2_Capacitor_SMD:C_0603; symbol Device:C_Small -> V2_Device:C_0603_10u; Manufacturer (none) -> TDK; Mouser (none) -> 810-C1608X6S1A106M; Product (none) -> C1608X6S1A106M080AC; Rating (none) -> 10V
- C105: renamed from C111; footprint Capacitor_SMD:C_0603_1608Metric -> V2_Capacitor_SMD:C_0603; symbol Device:C_Small -> V2_Device:C_0603_0u022; Manufacturer (none) -> YAGEO; Mouser (none) -> 603-CC603KPX7R9BB223; Product (none) -> CC0603KPX7R9BB223
- C106: renamed from C112; footprint Capacitor_SMD:C_0603_1608Metric -> V2_Capacitor_SMD:C_0603; symbol Device:C_Small -> V2_Device:C_0603_0u022; Manufacturer (none) -> YAGEO; Mouser (none) -> 603-CC603KPX7R9BB223; Product (none) -> CC0603KPX7R9BB223
- C107: renamed from C102; footprint Capacitor_SMD:C_0603_1608Metric -> V2_Capacitor_SMD:C_0603; symbol Device:C_Small -> V2_Device:C_0603_0u1; Manufacturer (none) -> TDK; Mouser (none) -> 810-CGA3E2X7R1H104MA; Product (none) -> CGA3E2X7R1H104M080AA; Rating (none) -> 50V
- C108: renamed from C103; footprint Capacitor_SMD:C_0603_1608Metric -> V2_Capacitor_SMD:C_0603; symbol Device:C_Small -> V2_Device:C_0603_0u1; Manufacturer (none) -> TDK; Mouser (none) -> 810-CGA3E2X7R1H104MA; Product (none) -> CGA3E2X7R1H104M080AA; Rating (none) -> 50V
- C109: renamed from C104; footprint Capacitor_SMD:C_0603_1608Metric -> V2_Capacitor_SMD:C_0603; symbol Device:C_Small -> V2_Device:C_0603_0u1; Manufacturer (none) -> TDK; Mouser (none) -> 810-CGA3E2X7R1H104MA; Product (none) -> CGA3E2X7R1H104M080AA; Rating (none) -> 50V
- C110: renamed from C105; footprint Capacitor_SMD:C_0603_1608Metric -> V2_Capacitor_SMD:C_0603; symbol Device:C_Small -> V2_Device:C_0603_0u1; Manufacturer (none) -> TDK; Mouser (none) -> 810-CGA3E2X7R1H104MA; Product (none) -> CGA3E2X7R1H104M080AA; Rating (none) -> 50V
- C111: renamed from C106; footprint Capacitor_SMD:C_0603_1608Metric -> V2_Capacitor_SMD:C_0603; symbol Device:C_Small -> V2_Device:C_0603_0u1; Manufacturer (none) -> TDK; Mouser (none) -> 810-CGA3E2X7R1H104MA; Product (none) -> CGA3E2X7R1H104M080AA; Rating (none) -> 50V
- C112: renamed from C107; footprint Capacitor_SMD:C_0603_1608Metric -> V2_Capacitor_SMD:C_0805; symbol Device:C_Small -> V2_Device:C_0805_10u; Manufacturer (none) -> TDK; Mouser (none) -> 810-C2012X5R1E106K; Product (none) -> C2012X5R1E106K125AB; Rating (none) -> 25V
- C113: renamed from C108; footprint Capacitor_SMD:C_0603_1608Metric -> V2_Capacitor_SMD:C_0805; symbol Device:C_Small -> V2_Device:C_0805_10u; Manufacturer (none) -> TDK; Mouser (none) -> 810-C2012X5R1E106K; Product (none) -> C2012X5R1E106K125AB; Rating (none) -> 25V
- D101: footprint LED_SMD:LED_0603_1608Metric -> V2_LED:LED_0603; symbol Device:LED_Small -> V2_Device:LED_0603_Orange; Manufacturer (none) -> ROHM Semiconductor; Mouser (none) -> 755-SML-D12D1WT86; Product (none) -> SML-D12D1WT86
- D102, D103: LCSC (none) -> C965555; Manufacturer (none) -> Worldsemi; Product (none) -> WS2812B-2020
- ESD101: Manufacturer (none) -> Semtech; Mouser (none) -> 947-RCLAMP0582N.TCT; Product (none) -> RCLAMP0582N.TCT
- FB101: value 47R -> 47 Ohm; symbol Device:FerriteBead_Small -> V2_Device:FerriteBead_3.1x5.1_47Ohm; Manufacturer (none) -> Fair-Rite; Mouser (none) -> 623-2743019447LF; Product (none) -> 2743019447
- FID101, FID102, FID103: value Fiducial -> Fiducial_Paste
- H101: value MountingHole_2mm -> 2mm
- H102: renamed from H103; value MountingHole_2mm -> 2mm
- H103: renamed from H105; value MountingHole_2mm -> 2mm
- H104: renamed from H106; value MountingHole_2mm -> 2mm
- H105: renamed from H102; value MountingHole_3mm -> 3mm
- H106: renamed from H104; value MountingHole_3mm -> 3mm
- INFO101: renamed from INFO102; value ORDER-NUMBER -> ~; footprint V2_Production:Order_Number -> V2_Production:Revision; symbol V2_Production:Order_Number -> V2_Production:Revision
- J101: renamed from J102; value WAGO-2065 -> WAGO 2065-100; Manufacturer (none) -> WAGO; Product (none) -> 2065-100/998-403
- J102: renamed from J105; value WAGO-2065 -> WAGO 2065-100; Manufacturer (none) -> WAGO; Product (none) -> 2065-100/998-403
- J103: renamed from J101; value CORTEX-DEBUG -> Cortex; footprint V2_Cortex_Debug:Cortex_Debug_Pad -> V2_Connector_Debug:Cortex; symbol V2_Cortex_Debug:Cortex_Debug -> V2_Connector_Debug:Cortex
- J104: renamed from J103; value WAGO-2065 -> WAGO 2065-100; Manufacturer (none) -> WAGO; Product (none) -> 2065-100/998-403
- J105: renamed from J104; value WAGO-2065 -> WAGO 2065-100; Manufacturer (none) -> WAGO; Product (none) -> 2065-100/998-403
- J106, J107: value WAGO-2065 -> WAGO 2065-100; Manufacturer (none) -> WAGO; Product (none) -> 2065-100/998-403
- R101: renamed from R105; footprint Resistor_SMD:R_0603_1608Metric -> V2_Resistor_SMD:R_0603; symbol Device:R_Small -> V2_Device:R_0603_100k; Manufacturer (none) -> Vishay; Mouser (none) -> 71-CRCW0603100KFKEAC; Product (none) -> CRCW0603100KFKEAC; Rating (none) -> 100mW
- R102: renamed from R108; footprint Resistor_SMD:R_0603_1608Metric -> V2_Resistor_SMD:R_0603; symbol Device:R_Small -> V2_Device:R_0603_10k; Manufacturer (none) -> Vishay; Mouser (none) -> 71-CRCW060310K0FKEAC; Product (none) -> CRCW060310K0FKEAC; Rating (none) -> 100mW
- R103: renamed from R106; footprint Resistor_SMD:R_0603_1608Metric -> V2_Resistor_SMD:R_0603; symbol Device:R_Small -> V2_Device:R_0603_10k; Manufacturer (none) -> Vishay; Mouser (none) -> 71-CRCW060310K0FKEAC; Product (none) -> CRCW060310K0FKEAC; Rating (none) -> 100mW
- R104: renamed from R102; footprint Resistor_SMD:R_0603_1608Metric -> V2_Resistor_SMD:R_0603; symbol Device:R_Small -> V2_Device:R_0603_100k; Manufacturer (none) -> Vishay; Mouser (none) -> 71-CRCW0603100KFKEAC; Product (none) -> CRCW0603100KFKEAC; Rating (none) -> 100mW
- R105: renamed from R103; footprint Resistor_SMD:R_0603_1608Metric -> V2_Resistor_SMD:R_0603; symbol Device:R_Small -> V2_Device:R_0603_2k7; Manufacturer (none) -> Vishay; Mouser (none) -> 71-CRCW06032K70FKEAC; Product (none) -> CRCW06032K70FKEAC; Rating (none) -> 100mW
- R106: renamed from R104; footprint Resistor_SMD:R_0603_1608Metric -> V2_Resistor_SMD:R_0603; symbol Device:R_Small -> V2_Device:R_0603_2k7; Manufacturer (none) -> Vishay; Mouser (none) -> 71-CRCW06032K70FKEAC; Product (none) -> CRCW06032K70FKEAC; Rating (none) -> 100mW
- R107: footprint Resistor_SMD:R_0603_1608Metric -> V2_Resistor_SMD:R_0603; symbol Device:R_Small -> V2_Device:R_0603_100k; Manufacturer (none) -> Vishay; Mouser (none) -> 71-CRCW0603100KFKEAC; Product (none) -> CRCW0603100KFKEAC; Rating (none) -> 100mW
- R108: renamed from R101; footprint Resistor_SMD:R_0603_1608Metric -> V2_Resistor_SMD:R_0603; symbol Device:R_Small -> V2_Device:R_0603_330R; Manufacturer (none) -> Vishay; Mouser (none) -> 71-CRCW0603330RFKEAC; Product (none) -> CRCW0603330RFKEAC; Rating (none) -> 100mW
- SW101: renamed from SW102; value SW_Push -> SKSG; symbol Switch:SW_Push -> V2_Switch:SKSG; Manufacturer (none) -> Alps Alpine; Mouser (none) -> 688-SKSGACE010; Product (none) -> SKSGACE010
- SW102: renamed from SW101; value SW_Push -> SKSG; symbol Switch:SW_Push -> V2_Switch:SKSG; Manufacturer (none) -> Alps Alpine; Mouser (none) -> 688-SKSGACE010; Product (none) -> SKSGACE010
- TVS101: renamed from TVS102; value SMAJ24CA -> SMBJ24CA; footprint Diode_SMD:D_SMA -> V2_Diode_SMD:D_SMB; symbol V2_Diode:SMAJ24CA -> V2_Diode:SMBJ24CA; Manufacturer (none) -> Bourns; Mouser (none) -> 652-SMBJ24CA-Q; Product (none) -> SMBJ24CA-Q; Rating (none) -> 24V
- TVS102: renamed from TVS101; footprint Diode_SMD:D_0603_1608Metric -> V2_Diode_SMD:D_0603; Manufacturer (none) -> Bourns; Mouser (none) -> 652-CG0603MLC-05LE; Product (none) -> CG0603MLC-05LE; Rating (none) -> 5V
- U101: renamed from U102; Manufacturer (none) -> Microchip Technology; Mouser (none) -> 556-ATSAMD51J19AMU; Product (none) -> ATSAMD51J19A-MU
- U102: renamed from U101; Manufacturer (none) -> Texas Instruments; Mouser (none) -> 595-TPS78433QWDRBRQ1; Product (none) -> TPS78433QWDRBRQ1
- Y101: symbol Device:Crystal_Small -> V2_Device:Crystal_3.2x1.5_32k768; Manufacturer (none) -> ABRACON; Mouser (none) -> 815-ABS0716632.768KT; Product (none) -> ABS07-166-32.768KHZ-T
- renumbered ICON108 to ICON101, ICON107 to ICON102, ICON101 to ICON103, ICON102 to ICON105, ICON105 to ICON106, ICON103 to ICON107, ICON106 to ICON108, INFO101 to INFO102
Connections:
- net Supply +24V renamed +24V-Supply
Other:
- moved on the sheet: C103, C105, C106, ESD101, FB101, FID101, FID102, FID103, H101, H102, H103, H104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

Commit message: Update Library
Parts:
- C101, C102: symbol V2_Device:C_0603_18p -> V2_Capacitor:0603_18p
- C103, C107, C108, C109, C110, C111: symbol V2_Device:C_0603_0u1 -> V2_Capacitor:0603_0u1
- C104: symbol V2_Device:C_0603_10u -> V2_Capacitor:0603_10u
- C105, C106: symbol V2_Device:C_0603_0u022 -> V2_Capacitor:0603_0u022
- C112, C113: symbol V2_Device:C_0805_10u -> V2_Capacitor:0805_10u
- D101: symbol V2_Device:LED_0603_Orange -> V2_LED:0603_Orange
- FB101: value 47 Ohm -> ~; symbol V2_Device:FerriteBead_3.1x5.1_47Ohm -> V2_Inductor:FerriteBead_3.1x5.1_47Ohm
- R101, R104, R107: symbol V2_Device:R_0603_100k -> V2_Resistor:0603_100k
- R102, R103: symbol V2_Device:R_0603_10k -> V2_Resistor:0603_10k
- R105, R106: symbol V2_Device:R_0603_2k7 -> V2_Resistor:0603_2k7
- R108: symbol V2_Device:R_0603_330R -> V2_Resistor:0603_330R
- Y101: symbol V2_Device:Crystal_3.2x1.5_32k768 -> V2_Crystal:3.2x1.5_32k768

Commit message: Update
Parts:
- FB101: value ~ -> 47 Ω
Connections:
- net Power is gone; now on net +24V-Supply: C106.1, FB101.2, R101.1
- net +24V-Supply: no longer C105.1, FB101.1, J101.1, TVS101.2 (A)
- new net +24V: C105.1, FB101.1, J101.1, TVS101.2 (A)
Other:
- moved on the sheet: J105, J106, J107
Changed lines of the file:
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@@
 	(wire
 		(pts
-			(xy 19.05 173.99) (xy 25.4 173.99)
+			(xy 19.05 173.99) (xy 33.02 173.99)
 		)
 		(stroke
@@
 		)
 	)
-	(label "Power"
+	(label "+24V-Supply"
 		(at 90.17 148.59 0)
 		(effects
@@
 		)
 	)
-	(label "+24V-Supply"
+	(label "+24V"
 		(at 41.91 148.59 0)
 		(effects
@@
 		)
 	)
-	(label "Power"
-		(at 25.4 173.99 180)
+	(label "+24V-Supply"
+		(at 33.02 173.99 180)
 		(effects
 			(font
@@
 			)
 		)
-		(property "Value" "~"
-			(at 75.184 154.559 90)
+		(property "Value" "47 Ω"
+			(at 72.898 154.559 90)
 			(effects
 				(font
@@
 		(at 236.22 142.24 0)
 		(unit 1)
-		(exclude_from_sim no)
+		(exclude_from_sim yes)
 		(in_bom no)
 		(on_board yes)
@@
 			)
 		)
-		(property "Sim.Enable" "0"
-			(at 236.22 142.24 0)
-			(effects
-				(font
-					(size 1.27 1.27)
-				)
-				(hide yes)
-			)
-		)
 		(instances
 			(project ""
@@
 		(at 236.22 161.29 0)
 		(unit 1)
-		(exclude_from_sim no)
+		(exclude_from_sim yes)
 		(in_bom no)
 		(on_board yes)
@@
 			)
 		)
-		(property "Sim.Enable" "0"
-			(at 236.22 161.29 0)
-			(effects
-				(font
-					(size 1.27 1.27)
-				)
-				(hide yes)
-			)
-		)
 		(instances
 			(project "wave"
@@
 		(at 236.22 154.94 0)
 		(unit 1)
-		(exclude_from_sim no)
+		(exclude_from_sim yes)
 		(in_bom no)
 		(on_board yes)
@@
 			)
 		)
-		(property "Sim.Enable" "0"
-			(at 236.22 154.94 0)
-			(effects
-				(font
-					(size 1.27 1.27)
-				)
-				(hide yes)
-			)
-		)
 		(instances
 			(project "wave"
@@
 		(at 175.26 160.02 0)
 		(unit 1)
-		(exclude_from_sim no)
+		(exclude_from_sim yes)
 		(in_bom no)
 		(on_board yes)
@@
 			)
 		)
-		(property "Sim.Enable" "0"
-			(at 175.26 160.02 0)
-			(effects
-				(font
-					(size 1.27 1.27)
-				)
-				(hide yes)
-			)
-		)
 		(instances
 			(project "wave"
@@
 		(at 203.835 152.4 0)
 		(unit 1)
-		(exclude_from_sim no)
+		(exclude_from_sim yes)
 		(in_bom no)
 		(on_board yes)
@@
 			)
 		)
-		(property "Sim.Enable" "0"
-			(at 203.835 152.4 0)
-			(effects
-				(font
-					(size 1.27 1.27)
-				)
-				(hide yes)
-			)
-		)
 		(instances
 			(project "wave"
@@
 		(at 236.22 148.59 0)
 		(unit 1)
-		(exclude_from_sim no)
+		(exclude_from_sim yes)
 		(in_bom no)
 		(on_board yes)
@@
 			)
 		)
-		(property "Sim.Enable" "0"
-			(at 236.22 148.59 0)
-			(effects
-				(font
-					(size 1.27 1.27)
-				)
-				(hide yes)
-			)
-		)
 		(instances
 			(project ""
@@
 	(symbol
 		(lib_id "V2_Connector_WAGO:2065")
-		(at 133.35 158.75 0)
+		(at 133.35 163.83 0)
 		(unit 1)
 		(exclude_from_sim no)
@@
 		(dnp no)
 		(property "Reference" "J107"
-			(at 134.62 161.544 0)
+			(at 134.62 163.83 0)
 			(effects
 				(font
@@
 		)
 		(property "Value" "WAGO 2065-100"
-			(at 143.256 164.084 0)
+			(at 143.256 166.37 0)
 			(effects
 				(font
@@
 		)
 		(property "Footprint" "V2_Connector_WAGO:2065-100"
-			(at 133.35 162.56 0)
+			(at 133.35 167.64 0)
 			(effects
 				(font
@@
 		)
 		(property "Datasheet" ""
-			(at 133.35 162.56 0)
+			(at 133.35 167.64 0)
 			(effects
 				(font
@@
 		)
 		(property "Description" ""
-			(at 133.35 158.75 0)
+			(at 133.35 163.83 0)
 			(effects
 				(font
@@
 		)
 		(property "Manufacturer" "WAGO"
-			(at 133.35 171.958 0)
+			(at 133.35 177.038 0)
 			(effects
 				(font
@@
 		)
 		(property "Product" "2065-100/998-403"
-			(at 133.35 175.26 0)
+			(at 133.35 180.34 0)
 			(effects
 				(font
@@
 		(at 236.22 167.64 0)
 		(unit 1)
-		(exclude_from_sim no)
+		(exclude_from_sim yes)
 		(in_bom no)
 		(on_board yes)
@@
 			)
 		)
-		(property "Sim.Enable" "0"
-			(at 236.22 167.64 0)
-			(effects
-				(font
-					(size 1.27 1.27)
-				)
-				(hide yes)
-			)
-		)
 		(instances
 			(project "wave"
@@
 		(at 203.835 161.925 0)
 		(unit 1)
-		(exclude_from_sim no)
+		(exclude_from_sim yes)
 		(in_bom no)
 		(on_board yes)
@@
 			)
 		)
-		(property "Sim.Enable" "0"
-			(at 203.835 161.925 0)
-			(effects
-				(font
-					(size 1.27 1.27)
-				)
-				(hide yes)
-			)
-		)
 		(instances
 			(project "wave"
@@
 		(dnp no)
 		(property "Reference" "J104"
-			(at 134.874 145.796 0)
+			(at 134.62 148.59 0)
 			(effects
 				(font
@@
 		)
 		(property "Value" "WAGO 2065-100"
-			(at 143.002 148.59 0)
+			(at 142.748 151.384 0)
 			(effects
 				(font
@@
 		(at 236.22 173.99 0)
 		(unit 1)
-		(exclude_from_sim no)
+		(exclude_from_sim yes)
 		(in_bom no)
 		(on_board yes)
@@
 			)
 		)
-		(property "Sim.Enable" "0"
-			(at 236.22 173.99 0)
-			(effects
-				(font
-					(size 1.27 1.27)
-				)
-				(hide yes)
-			)
-		)
 		(instances
 			(project "wave"
@@
 	(symbol
 		(lib_id "V2_Connector_WAGO:2065")
-		(at 133.35 151.13 0)
+		(at 133.35 153.67 0)
 		(unit 1)
 		(exclude_from_sim no)
@@
 		(dnp no)
 		(property "Reference" "J105"
-			(at 134.62 151.13 0)
+			(at 134.62 153.67 0)
 			(effects
 				(font
@@
 		)
 		(property "Value" "WAGO 2065-100"
-			(at 143.002 153.67 0)
+			(at 143.002 156.21 0)
 			(effects
 				(font
@@
 		)
 		(property "Footprint" "V2_Connector_WAGO:2065-100"
-			(at 133.35 154.94 0)
+			(at 133.35 157.48 0)
 			(effects
 				(font
@@
 		)
 		(property "Datasheet" ""
-			(at 133.35 154.94 0)
+			(at 133.35 157.48 0)
 			(effects
 				(font
@@
 		)
 		(property "Description" ""
-			(at 133.35 151.13 0)
+			(at 133.35 153.67 0)
 			(effects
 				(font
@@
 		)
 		(property "Manufacturer" "WAGO"
-			(at 133.35 164.338 0)
+			(at 133.35 166.878 0)
 			(effects
 				(font
@@
 		)
 		(property "Product" "2065-100/998-403"
-			(at 133.35 167.64 0)
+			(at 133.35 170.18 0)
 			(effects
 				(font
@@
 	(symbol
 		(lib_id "V2_Connector_WAGO:2065")
-		(at 133.35 156.21 0)
+		(at 133.35 158.75 0)
 		(unit 1)
 		(exclude_from_sim no)
@@
 		(dnp no)
 		(property "Reference" "J106"
-			(at 134.62 156.21 0)
+			(at 134.62 158.75 0)
 			(effects
 				(font
@@
 		)
 		(property "Value" "WAGO 2065-100"
-			(at 143.002 159.004 0)
+			(at 143.002 161.544 0)
 			(effects
 				(font
@@
 		)
 		(property "Footprint" "V2_Connector_WAGO:2065-100"
-			(at 133.35 160.02 0)
+			(at 133.35 162.56 0)
 			(effects
 				(font
@@
 		)
 		(property "Datasheet" ""
-			(at 133.35 160.02 0)
+			(at 133.35 162.56 0)
 			(effects
 				(font
@@
 		)
 		(property "Description" ""
-			(at 133.35 156.21 0)
+			(at 133.35 158.75 0)
 			(effects
 				(font
@@
 		)
 		(property "Manufacturer" "WAGO"
-			(at 133.35 169.418 0)
+			(at 133.35 171.958 0)
 			(effects
 				(font
@@
 		)
 		(property "Product" "2065-100/998-403"
-			(at 133.35 172.72 0)
+			(at 133.35 175.26 0)
 			(effects
 				(font
@@
 		(at 203.835 172.72 0)
 		(unit 1)
-		(exclude_from_sim no)
+		(exclude_from_sim yes)
 		(in_bom no)
 		(on_board yes)
@@
 			)
 		)
-		(property "Sim.Enable" "0"
-			(at 203.835 172.72 0)
-			(effects
-				(font
-					(size 1.27 1.27)
-				)
-				(hide yes)
-			)
-		)
 		(instances
 			(project "wave"
@@
 		)
 		(pin "OUT1P" output
-			(at 128.27 156.21 0)
+			(at 128.27 158.75 0)
 			(effects
 				(font
@@
 		)
 		(pin "OUT1N" output
-			(at 128.27 158.75 0)
+			(at 128.27 163.83 0)
 			(effects
 				(font
@@
 		)
 		(pin "OUT0N" output
-			(at 128.27 151.13 0)
+			(at 128.27 153.67 0)
 			(effects
 				(font
