File: hardware/wave.kicad_sch (KiCad schematic)
At the start: 62 parts, among them J101 WAGO 2065-100, J102 WAGO 2065-100, J103 Cortex, J104 WAGO 2065-100, J105 WAGO 2065-100, J106 WAGO 2065-100, J107 WAGO 2065-100, SW101 SKSG, SW102 SKSG, U101 ATSAMD51J, U102 TPS78433QWDRBRQ1, Y101 32k768

Commit message: Update power routing
Parts:
- D101: footprint V2_LED:LED_0603 -> V2_LED:LED_1608
- INFO102: value Layer_Numbers -> Layer_Numbers-4; footprint V2_Production:Layer_Numbers -> V2_Production:Layer_Numbers-4; symbol V2_Production:Layer_Numbers -> V2_Production:Layer_Numbers-4
- TVS102: footprint V2_Diode_SMD:D_0603 -> V2_Diode_SMD:D_1608
Connections:
- net USB+: now also ESD101.3 (D1)
- net USB-: now also ESD101.2 (D2)
- no-connect marks 29 -> 27
