File: hardware/LinkPlug.kicad_sch (KiCad schematic)
At the start: 4 parts, among them J301 2x05_Horizontal, U301 THVD2442

Commit message: Refresh
Other:
- title: V2 Link -> V2 wave

Commit message: Update
Parts:
- C301: Id (none) -> Capacitor:${SYMBOL_NAME}
- J301: Id (none) -> Header:${SYMBOL_NAME}
- R301: Id (none) -> Resistor:${SYMBOL_NAME}
- U301: Id (none) -> RS485:${SYMBOL_NAME}
Changed lines of the file:
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@@
 	(title_block
 		(title "V2 wave")
-		(date "2026-03-26")
-		(rev "2026-03-11")
+		(date "2026-04-03")
+		(rev "2026-04-03")
 		(company "Plug")
 	)
@@
 			)
 		)
+		(property "Id" "RS485:${SYMBOL_NAME}"
+			(at 146.05 109.22 0)
+			(hide yes)
+			(show_name no)
+			(do_not_autoplace no)
+			(effects
+				(font
+					(size 1.27 1.27)
+				)
+			)
+		)
 		(pin "1"
 		)
@@
 			)
 		)
+		(property "Id" "Resistor:${SYMBOL_NAME}"
+			(at 157.48 86.36 0)
+			(hide yes)
+			(show_name no)
+			(do_not_autoplace no)
+			(effects
+				(font
+					(size 1.27 1.27)
+				)
+			)
+		)
 		(pin "1"
 		)
@@
 			)
 		)
+		(property "Id" "Header:${SYMBOL_NAME}"
+			(at 146.05 144.78 0)
+			(hide yes)
+			(show_name no)
+			(do_not_autoplace no)
+			(effects
+				(font
+					(size 1.27 1.27)
+				)
+			)
+		)
 		(pin "1"
 		)
@@
 			(hide yes)
 			(show_name no)
+			(do_not_autoplace no)
+			(effects
+				(font
+					(size 1.27 1.27)
+				)
+			)
+		)
+		(property "Id" "Capacitor:${SYMBOL_NAME}"
+			(at 137.16 72.39 0)
+			(hide yes)
+			(show_name no)

Commit message: Update
Parts:
- J301: Rating (none) -> 1A
- U301: Rating (none) -> 20Mbps
Other:
- company: Plug -> Versio Duo
Changed lines of the file:
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@@
 	(title_block
 		(title "V2 wave")
-		(date "2026-04-03")
-		(rev "2026-04-03")
-		(company "Plug")
+		(date "2026-04-14")
+		(rev "2026-04-14")
+		(company "Versio Duo")
+		(comment 1 "Power Amplifier")
 	)
 	(rectangle
@@
 		(in_pos_files yes)
 		(dnp no)
-		(property "Reference" "#PWR309"
+		(property "Reference" "#PWR301"
 			(at 137.16 66.04 0)
 			(hide yes)
@@
 			(project "wave"
 				(path "/6c8448b4-b04d-47e1-934e-e40cbe27a7be/c6db2f80-f80f-4104-8ca1-02f0ab85cfea"
-					(reference "#PWR309")
+					(reference "#PWR301")
 					(unit 1)
 				)
@@
 			)
 		)
+		(property "Rating" "20Mbps"
+			(at 147.32 116.84 0)
+			(hide yes)
+			(show_name no)
+			(do_not_autoplace no)
+			(effects
+				(font
+					(size 1.27 1.27)
+				)
+			)
+		)
 		(pin "1"
 		)
@@
 			)
 		)
+		(property "Rating" "1A"
+			(at 146.05 160.02 0)
+			(hide yes)
+			(show_name no)
+			(do_not_autoplace no)
+			(effects
+				(font
+					(size 1.27 1.27)
+				)
+			)
+		)
 		(pin "1"
 		)
@@
 		(in_pos_files yes)
 		(dnp no)
-		(property "Reference" "#PWR305"
+		(property "Reference" "#PWR306"
 			(at 143.51 149.86 0)
 			(hide yes)
@@
 			(project "wave"
 				(path "/6c8448b4-b04d-47e1-934e-e40cbe27a7be/c6db2f80-f80f-4104-8ca1-02f0ab85cfea"
-					(reference "#PWR305")
+					(reference "#PWR306")
 					(unit 1)
 				)
@@
 		(in_pos_files yes)
 		(dnp no)
-		(property "Reference" "#PWR301"
+		(property "Reference" "#PWR302"
 			(at 133.35 127 0)
 			(hide yes)
@@
 			(project "wave"
 				(path "/6c8448b4-b04d-47e1-934e-e40cbe27a7be/c6db2f80-f80f-4104-8ca1-02f0ab85cfea"
-					(reference "#PWR301")
+					(reference "#PWR302")
 					(unit 1)
 				)
@@
 		(in_pos_files yes)
 		(dnp no)
-		(property "Reference" "#PWR302"
+		(property "Reference" "#PWR303"
 			(at 143.51 132.08 0)
 			(hide yes)
@@
 			(project "wave"
 				(path "/6c8448b4-b04d-47e1-934e-e40cbe27a7be/c6db2f80-f80f-4104-8ca1-02f0ab85cfea"
-					(reference "#PWR302")
+					(reference "#PWR303")
 					(unit 1)
 				)
@@
 		(in_pos_files yes)
 		(dnp no)
-		(property "Reference" "#PWR304"
+		(property "Reference" "#PWR305"
 			(at 146.05 99.06 0)
 			(hide yes)
@@
 			(project "wave"
 				(path "/6c8448b4-b04d-47e1-934e-e40cbe27a7be/c6db2f80-f80f-4104-8ca1-02f0ab85cfea"
-					(reference "#PWR304")
+					(reference "#PWR305")
 					(unit 1)
 				)
@@
 		(in_pos_files yes)
 		(dnp no)
-		(property "Reference" "#PWR307"
+		(property "Reference" "#PWR308"
 			(at 148.59 127 0)
 			(hide yes)
@@
 			(project "wave"
 				(path "/6c8448b4-b04d-47e1-934e-e40cbe27a7be/c6db2f80-f80f-4104-8ca1-02f0ab85cfea"
-					(reference "#PWR307")
+					(reference "#PWR308")
 					(unit 1)
 				)
@@
 		(in_pos_files yes)
 		(dnp no)
-		(property "Reference" "#PWR303"
+		(property "Reference" "#PWR304"
 			(at 146.05 58.42 0)
 			(hide yes)
@@
 			(project "wave"
 				(path "/6c8448b4-b04d-47e1-934e-e40cbe27a7be/c6db2f80-f80f-4104-8ca1-02f0ab85cfea"
-					(reference "#PWR303")
+					(reference "#PWR304")
 					(unit 1)
 				)
@@
 		(in_pos_files yes)
 		(dnp no)
-		(property "Reference" "#PWR306"
+		(property "Reference" "#PWR307"
 			(at 153.67 153.67 0)
 			(hide yes)
@@
 			(project "wave"
 				(path "/6c8448b4-b04d-47e1-934e-e40cbe27a7be/c6db2f80-f80f-4104-8ca1-02f0ab85cfea"
-					(reference "#PWR306")
+					(reference "#PWR307")
 					(unit 1)
 				)
@@
 		(in_pos_files yes)
 		(dnp no)
-		(property "Reference" "#PWR308"
+		(property "Reference" "#PWR309"
 			(at 158.75 132.08 0)
 			(hide yes)
@@
 			(project "wave"
 				(path "/6c8448b4-b04d-47e1-934e-e40cbe27a7be/c6db2f80-f80f-4104-8ca1-02f0ab85cfea"
-					(reference "#PWR308")
+					(reference "#PWR309")
 					(unit 1)
 				)

Commit message: Good Bye Imperial
Parts:
- C301: footprint V2_Capacitor_SMD:C_0603 -> V2_Capacitor_SMD:C_1608; symbol V2_Capacitor:0603_0u1 -> V2_Capacitor:1608_0u1
- R301: footprint V2_Resistor_SMD:R_0603 -> V2_Resistor_SMD:R_1608; symbol V2_Resistor:0603_100R -> V2_Resistor:1608_100R
Changed lines of the file:
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@@
 	)
 	(symbol
-		(lib_id "V2_Resistor:0603_100R")
+		(lib_id "V2_Resistor:1608_100R")
 		(at 157.48 72.39 0)
 		(unit 1)
@@
 			)
 		)
-		(property "Footprint" "V2_Resistor_SMD:R_0603"
+		(property "Footprint" "V2_Resistor_SMD:R_1608"
 			(at 157.48 88.138 0)
 			(hide yes)
@@
 	)
 	(symbol
-		(lib_id "V2_Capacitor:0603_0u1")
+		(lib_id "V2_Capacitor:1608_0u1")
 		(at 137.16 57.15 0)
 		(unit 1)
@@
 			)
 		)
-		(property "Footprint" "V2_Capacitor_SMD:C_0603"
+		(property "Footprint" "V2_Capacitor_SMD:C_1608"
 			(at 137.16 57.15 0)
 			(hide yes)
