File: hardware/LinkSocket.kicad_sch (KiCad schematic)
At the start: 4 parts, among them J401 2x05_Horizontal, U401 THVD2442

Commit message: Refresh
Other:
- title: V2 Link -> V2 wave

Commit message: Update
Parts:
- C401: Id (none) -> Capacitor:${SYMBOL_NAME}
- J401: Id (none) -> Header:${SYMBOL_NAME}
- R401: Id (none) -> Resistor:${SYMBOL_NAME}
- U401: Id (none) -> RS485:${SYMBOL_NAME}
Changed lines of the file:
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@@
 	(title_block
 		(title "V2 wave")
-		(date "2026-03-26")
-		(rev "2026-03-11")
+		(date "2026-04-03")
+		(rev "2026-04-03")
 		(company "Socket")
 	)
@@
 			)
 		)
+		(property "Id" "RS485:${SYMBOL_NAME}"
+			(at 153.67 119.38 0)
+			(hide yes)
+			(show_name no)
+			(do_not_autoplace no)
+			(effects
+				(font
+					(size 1.27 1.27)
+				)
+			)
+		)
 		(pin "1"
 		)
@@
 			)
 		)
+		(property "Id" "Resistor:${SYMBOL_NAME}"
+			(at 165.1 96.52 0)
+			(hide yes)
+			(show_name no)
+			(do_not_autoplace no)
+			(effects
+				(font
+					(size 1.27 1.27)
+				)
+			)
+		)
 		(pin "1"
 		)
@@
 			)
 		)
+		(property "Id" "Header:${SYMBOL_NAME}"
+			(at 153.67 158.75 0)
+			(hide yes)
+			(show_name no)
+			(do_not_autoplace no)
+			(effects
+				(font
+					(size 1.27 1.27)
+				)
+			)
+		)
 		(pin "1"
 		)
@@
 			(hide yes)
 			(show_name no)
+			(do_not_autoplace no)
+			(effects
+				(font
+					(size 1.27 1.27)
+				)
+			)
+		)
+		(property "Id" "Capacitor:${SYMBOL_NAME}"
+			(at 142.24 82.55 0)
+			(hide yes)
+			(show_name no)

Commit message: Update
Parts:
- J401: Rating (none) -> 1A
- U401: Rating (none) -> 20Mbps
Other:
- company: Socket -> Versio Duo
Changed lines of the file:
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@@
 	(title_block
 		(title "V2 wave")
-		(date "2026-04-03")
-		(rev "2026-04-03")
-		(company "Socket")
+		(date "2026-04-14")
+		(rev "2026-04-14")
+		(company "Versio Duo")
+		(comment 1 "Power Amplifier")
 	)
 	(junction
@@
 		(in_pos_files yes)
 		(dnp no)
-		(property "Reference" "#PWR403"
+		(property "Reference" "#PWR404"
 			(at 153.67 68.58 0)
 			(hide yes)
@@
 			(project "wave"
 				(path "/6c8448b4-b04d-47e1-934e-e40cbe27a7be/2a03ea79-269e-4abf-833c-000ba0ff13d7"
-					(reference "#PWR403")
+					(reference "#PWR404")
 					(unit 1)
 				)
@@
 			)
 		)
+		(property "Rating" "20Mbps"
+			(at 154.94 127 0)
+			(hide yes)
+			(show_name no)
+			(do_not_autoplace no)
+			(effects
+				(font
+					(size 1.27 1.27)
+				)
+			)
+		)
 		(pin "1"
 		)
@@
 		(in_pos_files yes)
 		(dnp no)
-		(property "Reference" "#PWR401"
+		(property "Reference" "#PWR402"
 			(at 140.97 140.97 0)
 			(hide yes)
@@
 			(project "wave"
 				(path "/6c8448b4-b04d-47e1-934e-e40cbe27a7be/2a03ea79-269e-4abf-833c-000ba0ff13d7"
-					(reference "#PWR401")
+					(reference "#PWR402")
 					(unit 1)
 				)
@@
 		(in_pos_files yes)
 		(dnp no)
-		(property "Reference" "#PWR404"
+		(property "Reference" "#PWR405"
 			(at 153.67 109.22 0)
 			(hide yes)
@@
 			(project "wave"
 				(path "/6c8448b4-b04d-47e1-934e-e40cbe27a7be/2a03ea79-269e-4abf-833c-000ba0ff13d7"
-					(reference "#PWR404")
+					(reference "#PWR405")
 					(unit 1)
 				)
@@
 		(in_pos_files yes)
 		(dnp no)
-		(property "Reference" "#PWR407"
+		(property "Reference" "#PWR401"
 			(at 142.24 76.2 0)
 			(hide yes)
@@
 			(project "wave"
 				(path "/6c8448b4-b04d-47e1-934e-e40cbe27a7be/2a03ea79-269e-4abf-833c-000ba0ff13d7"
-					(reference "#PWR407")
+					(reference "#PWR401")
 					(unit 1)
 				)
@@
 		(in_pos_files yes)
 		(dnp no)
-		(property "Reference" "#PWR406"
+		(property "Reference" "#PWR407"
 			(at 166.37 146.05 0)
 			(hide yes)
@@
 			(project "wave"
 				(path "/6c8448b4-b04d-47e1-934e-e40cbe27a7be/2a03ea79-269e-4abf-833c-000ba0ff13d7"
-					(reference "#PWR406")
+					(reference "#PWR407")
 					(unit 1)
 				)
@@
 			)
 		)
+		(property "Rating" "1A"
+			(at 153.67 173.99 0)
+			(hide yes)
+			(show_name no)
+			(do_not_autoplace no)
+			(effects
+				(font
+					(size 1.27 1.27)
+				)
+			)
+		)
 		(pin "1"
 		)
@@
 		(in_pos_files yes)
 		(dnp no)
-		(property "Reference" "#PWR402"
+		(property "Reference" "#PWR403"
 			(at 151.13 146.05 0)
 			(hide yes)
@@
 			(project "wave"
 				(path "/6c8448b4-b04d-47e1-934e-e40cbe27a7be/2a03ea79-269e-4abf-833c-000ba0ff13d7"
-					(reference "#PWR402")
+					(reference "#PWR403")
 					(unit 1)
 				)
@@
 		(in_pos_files yes)
 		(dnp no)
-		(property "Reference" "#PWR405"
+		(property "Reference" "#PWR406"
 			(at 156.21 140.97 0)
 			(hide yes)
@@
 			(project "wave"
 				(path "/6c8448b4-b04d-47e1-934e-e40cbe27a7be/2a03ea79-269e-4abf-833c-000ba0ff13d7"
-					(reference "#PWR405")
+					(reference "#PWR406")
 					(unit 1)
 				)

Commit message: Good Bye Imperial
Parts:
- C401: footprint V2_Capacitor_SMD:C_0603 -> V2_Capacitor_SMD:C_1608; symbol V2_Capacitor:0603_0u1 -> V2_Capacitor:1608_0u1
- R401: footprint V2_Resistor_SMD:R_0603 -> V2_Resistor_SMD:R_1608; symbol V2_Resistor:0603_100R -> V2_Resistor:1608_100R
Changed lines of the file:
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@@
 	)
 	(symbol
-		(lib_id "V2_Resistor:0603_100R")
+		(lib_id "V2_Resistor:1608_100R")
 		(at 165.1 82.55 0)
 		(unit 1)
@@
 			)
 		)
-		(property "Footprint" "V2_Resistor_SMD:R_0603"
+		(property "Footprint" "V2_Resistor_SMD:R_1608"
 			(at 165.1 98.298 0)
 			(hide yes)
@@
 	)
 	(symbol
-		(lib_id "V2_Capacitor:0603_0u1")
+		(lib_id "V2_Capacitor:1608_0u1")
 		(at 142.24 67.31 0)
 		(unit 1)
@@
 			)
 		)
-		(property "Footprint" "V2_Capacitor_SMD:C_0603"
+		(property "Footprint" "V2_Capacitor_SMD:C_1608"
 			(at 142.24 67.31 0)
 			(hide yes)
